Commit message: Update model.urdf

File: robotic_arm/model.urdf (robot description, URDF)
Before this commit: robot robotic_arm, 35 links, 34 joints
Links:
- link H1_F1_base_link: geometry collision mesh filename=package://robotic_arm/meshes/v2/finger_base_link_simple.dae; visual mesh filename=package://robotic_arm/meshes/v2/finger_base_link_simple.dae
- link H1_F1_link_1: geometry collision mesh filename=package://robotic_arm/meshes/v2/finger_prox_link_simple.dae; visual mesh filename=package://robotic_arm/meshes/v2/finger_prox_link_simple.dae
- link H1_F1_link_2: geometry collision mesh filename=package://robotic_arm/meshes/v2/finger_dist_link_simple.dae; visual mesh filename=package://robotic_arm/meshes/v2/finger_dist_link_simple.dae
- link H1_F1_palm_link: geometry visual mesh filename=package://robotic_arm/meshes/v2/finger_palm_link.dae
- link H1_F1_tip: geometry collision mesh filename=package://robotic_arm/meshes/omd-d18-tip.dae; visual mesh filename=package://robotic_arm/meshes/omd-d18-tip.dae
- link H1_F2_base_link: geometry collision mesh filename=package://robotic_arm/meshes/v2/finger_base_link_simple.dae; visual mesh filename=package://robotic_arm/meshes/v2/finger_base_link_simple.dae
- link H1_F2_link_1: geometry collision mesh filename=package://robotic_arm/meshes/v2/finger_prox_link_simple.dae; visual mesh filename=package://robotic_arm/meshes/v2/finger_prox_link_simple.dae
- link H1_F2_link_2: geometry collision mesh filename=package://robotic_arm/meshes/v2/finger_dist_link_simple.dae; visual mesh filename=package://robotic_arm/meshes/v2/finger_dist_link_simple.dae
- link H1_F2_palm_link: geometry visual mesh filename=package://robotic_arm/meshes/v2/finger_palm_link.dae
- link H1_F2_tip: geometry collision mesh filename=package://robotic_arm/meshes/omd-d18-tip.dae; visual mesh filename=package://robotic_arm/meshes/omd-d18-tip.dae
- link H1_F3_base_link: geometry collision mesh filename=package://robotic_arm/meshes/v2/finger_base_link_simple.dae; visual mesh filename=package://robotic_arm/meshes/v2/finger_base_link_simple.dae
- link H1_F3_link_1: geometry collision mesh filename=package://robotic_arm/meshes/v2/finger_prox_link_simple.dae; visual mesh filename=package://robotic_arm/meshes/v2/finger_prox_link_simple.dae
- link H1_F3_link_2: geometry collision mesh filename=package://robotic_arm/meshes/v2/finger_dist_link_simple.dae; visual mesh filename=package://robotic_arm/meshes/v2/finger_dist_link_simple.dae
- link H1_F3_palm_link: geometry visual mesh filename=package://robotic_arm/meshes/v2/finger_palm_link.dae
- link H1_F3_tip: geometry collision mesh filename=package://robotic_arm/meshes/omd-d18-tip.dae; visual mesh filename=package://robotic_arm/meshes/omd-d18-tip.dae
- link H1_base_link: geometry collision mesh filename=package://robotic_arm/meshes/v2/palm_link_simple.dae; visual mesh filename=package://robotic_arm/meshes/v2/palm_link_simple.dae

Commit message: Update model.urdf
Relocated robot base

File: robotic_arm/model.urdf (robot description, URDF)
Before this commit: robot robotic_arm, 35 links, 34 joints
Joints:
- joint world_joint: origin xyz=0.0 -1.0 1.0 rpy=0.0 0.0 0.0 -> xyz=0.0 -0.7 1.0 rpy=0.0 0.0 0.0
